Commit message: 切换到 4 自由度机械臂：模型/接口层按 6 自由度版本对齐
- arm_model/model：换成 4 自由度机械臂自己的几何/惯量/限位/网格（base_link 5.0 MB），
  URDF 补 xacro headless 参数与 <ros2_control>（effort 命令 + position/velocity/effort/
  acceleration 状态，mujoco_model 指向 model/scene.xml），网格路径从 kdl_tools 改到
  arm_model/model；MJCF 由 <position> 隐式伺服改为 <motor> 力矩执行器（ctrlrange ±50
  与 URDF effort 一致），关节显式 limited="true"；scene 显式 timestep=0.002 且开启
  地面接触。删除 6 自由度的 link5/link6、4 自由度遗留的 torque 变体与 model_2 备份。
- 控制器：末端坐标系参数化 end_effector_frame（auto_declare，默认 link6，YAML 设 link4），
  ModelFromURDF 与 measure 激励轨迹共用；启动日志打印实际生效值。
- 配置：joints/default_kp/default_kd/reset_joint_pos/admittance 改 4 关节；kp/kd 按 500 Hz
  显式力矩环重新整定（joint3 的 kd 必须 < 0.2，肩关节 kp 需压过重力 Hessian -6.4）；
  tasks.yaml 目标点改 4 维；measure 连杆间碰撞约束默认关闭（4 自由度 base_link 网格
  5 MB，开启时激励轨迹生成 >4.5 min），地面净空保留，measure step_timeout 留 600 s 余量。
- 验证：headless 仿真能加载 4 关节/4 motor，自动复位收敛；reset_then_joint 关节跟踪
  误差 0.0000 rad；arm_measure_sim 端到端跑通并产出 4 关节、5000 行 CSV（生成 ~46 s）。

File: src/arm_model/model/robotic_arm.urdf (robot description, URDF)
Before this commit: robot robotic_arm, 8 links, 7 joints
Links:
- removed link link5
- removed link link6
- link base_link: mass 1.0998 -> 0.445927939104524
- link link1: mass 2.34956808405639 -> 0.422761931253973
- link link2: mass 1.23727124080295 -> 0.352210008949705
- link link3: mass 0.370266089775016 -> 0.0763832349061947
- link link4: mass 1.54177209165349 -> 0.267547364804174
Joints:
- removed joint joint5
- removed joint joint6
- joint joint1: limit lower=-1.8 upper=1.8 effort=50 velocity=10 -> lower=-1.5708 upper=1.5708 effort=50 velocity=10; origin xyz=0 0 0 rpy=0 0 0 -> xyz=0 0.042 0.05 rpy=1.5708 -1.5708 0.0
- joint joint2: axis 0 0 1 -> 0 -1 0; limit lower=-1.570796327 upper=1.570796327 effort=50 velocity=10 -> lower=-3.1 upper=3.1 effort=50 velocity=10; origin xyz=0 0.03675 0.153 rpy=1.5708 -1.5708 0 -> xyz=0.374 0 0.0401 rpy=1.5708 0 0
- joint joint3: axis 0 0 1 -> 1 0 0; limit lower=-2.9 upper=2.9 effort=50 velocity=10 -> lower=-3.14 upper=3.14 effort=50 velocity=10; origin xyz=0.52 0 0.08565 rpy=0 0 0 -> xyz=0.4014 -0.0055 0 rpy=0 0 0
- joint joint4: limit lower=-2.0 upper=1.8 effort=50 velocity=10 -> lower=-1.5708 upper=1.5708 effort=50 velocity=10; origin xyz=0.436 0 0.0225 rpy=0 0 0 -> xyz=0.0430000000000001 -0.0199999999998909 0 rpy=1.5707963267949 0 3.14159265358979
